File: electronics/controller_board/controller_board.kicad_pcb (KiCad board)
At the start: 2 copper layers, 82 parts, among them P1 CONN_02X08, P10 Arietta G25, P11 Arietta G25 aux, P12 CONN_01X02, P13 USB_A, P2 CONN_01X08, P3 CONN_01X08, P4 CONN_02X08, P5 CONN_02X08, P6 CONN_01X08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

Commit message: More routing on board
Parts:
- removed P11: Arietta G25 aux, Pin_Headers:Pin_Header_Straight_2x20
- added REF**: Hole_3mm, custom_footprints:Hole_3mm, F.Cu at (156.8, 113.0)
- added m3: Hole_3mm, custom_footprints:Hole_3mm, F.Cu at (48.3, 113.0)
- P13: footprint Connect:USB_A_Vertical -> Connect:USB_A
- U1, U2: footprint Housings_SSOP:TSSOP-28_4.4x9.7mm_Pitch0.65mm -> custom_footprints:TSSOP-28
- U3: footprint Housings_DFN_QFN:DFN-18-1EP_4x5mm_Pitch0.5mm -> custom_footprints:bno055
- Y1: footprint Crystals:Crystal_HC49-SD_SMD -> Capacitors_SMD:C_0603
- moved R44 239.6 mm to (116.8, 95.9), turned to 90 degrees
- moved D2 219.2 mm to (136.5, 38.1)
- moved U3 217.3 mm to (102.9, 105.4), turned to 270 degrees
- moved U4 211.8 mm to (129.5, 52.7)
- moved C6 206.1 mm to (102.9, 99.1)
- moved Y1 177.9 mm to (107.3, 104.8), turned to 90 degrees
- moved D1 166.8 mm to (33.7, 67.3)
- moved R46 166.3 mm to (27.9, 67.3)
- moved C3 162.5 mm to (102.9, 101.0)
- moved C5 155.7 mm to (107.3, 98.4), turned to 90 degrees
- moved C4 146.0 mm to (109.2, 98.4), turned to 90 degrees
- moved C2 124.5 mm to (148.6, 113.0), turned to 270 degrees
- moved P12 115.7 mm to (97.8, 34.3)
- moved JP7 114.3 mm to (119.4, 102.2), turned to 270 degrees
- moved C7 112.3 mm to (74.9, 34.9)
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Connections:
- P13 pad 5: VCC -> GND
- U3 pad 11: Net-(P9-Pad4) -> Net-(P9-Pad3)
- U3 pad 14: Net-(P9-Pad3) -> Net-(P9-Pad4)
- U3 pad 5: Net-(P9-Pad2) -> Net-(P9-Pad1)
- U3 pad 6: Net-(P9-Pad1) -> Net-(P9-Pad2)
Routing:
- net Net-(R26-Pad2): track 0.00 -> 25.5 mm
- net Net-(R41-Pad2): track 0.00 -> 25.4 mm
- net Net-(R1-Pad1): track 0.00 -> 25.1 mm
- net Net-(R16-Pad1): track 0.00 -> 25.1 mm
- net Net-(R27-Pad2): track 0.00 -> 22.6 mm
- net Net-(R40-Pad2): track 0.00 -> 22.6 mm
- net Net-(R2-Pad1): track 0.00 -> 22.3 mm
- net Net-(R15-Pad1): track 0.00 -> 22.3 mm
- net Net-(R28-Pad2): track 0.00 -> 19.7 mm
- net Net-(R39-Pad2): track 0.00 -> 19.7 mm
- net Net-(R3-Pad1): track 0.00 -> 19.5 mm
- net Net-(R14-Pad1): track 0.00 -> 19.5 mm
- net Net-(R29-Pad2): track 0.00 -> 16.9 mm
- net Net-(R38-Pad2): track 0.00 -> 16.9 mm
- net Net-(R4-Pad1): track 0.00 -> 16.7 mm
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Other:
- board outline added: 118.7 x 55.9 mm
- net class Default: clearance 0.2 -> 0.17; trace_width 0.25 -> 0.35
- rule trace_clearance: 0.2 -> 0.17
- board text added: "S16"
- board text added: "S17"
- board text added: "S18"
- board text added: "S19"
- board text added: "S20"
- board text added: "S21"
- board text added: "S22"
- board text added: "S23"
- board text added: "S24"
- board text added: "S25"
- board text added: "S26"
- board text added: "S27"
- board text added: "S28"
- board text added: "S29"
- board text added: "S30"
- board text added: "S31"
